File: misc/final.brd (EAGLE design)
At the start: 160 x 100 mm, 7 parts, among them IC1 L293D

Commit message: Electric diagram + new tests
Parts:
- removed C1: 10uF, SparkFun-Capacitors:CPOL-RADIAL-2.5MM-5MM
- removed IC1: L293D, st-microelectronics:DIL16
- removed R1, R2: 1k, SparkFun-Resistors:AXIAL-0.3
- added CONN_DEANS: (no value), SparkFun-Connectors:DEANS
- added J3, MOTORS: (no value), SparkFun-Connectors:1X04
- added L293D: L293D, st-microelectronics:DIL16
- J1: device SparkFun-Connectors:1X16 -> SparkFun-Connectors:1X03
- J2: device SparkFun-Connectors:1X12 -> SparkFun-Connectors:1X09
- moved U$1 80.3 mm to (-20.3, 11.4)
- moved J1 79.1 mm to (-76.2, -22.9)
- moved J2 79.1 mm to (-76.2, -26.7)
Connections:
- removed net GND1: IC1.4
- removed net GND2: IC1.5
- removed net GND3: IC1.13
- removed net GND4: IC1.12
- removed net VCC1: IC1.16
- removed net VCC2: IC1.8
- new net EN1-2: L293D.1
- new net EN3-4: L293D.9
- new net GND: CONN_DEANS.-, L293D.12, L293D.13, L293D.4, L293D.5, U$1.GND
- new net GND-LEFT: L293D.6, MOTORS.3
- new net GND-RIGHT: L293D.11, MOTORS.2
- new net IN1: L293D.2
- new net IN2: L293D.7
- new net IN3: L293D.10
- new net IN4: L293D.15
- new net V+: CONN_DEANS.+, L293D.8, U$1.RAW
- new net VCC: L293D.16, U$1.5V
- new net VCC-LEFT: L293D.3, MOTORS.4
- new net VCC-RIGHT: L293D.14, MOTORS.1
