File: misc/final.sch (EAGLE design)
At the start: 13 parts

Commit message: Update schematic
Parts:
- removed L293D: L293D, st-microelectronics:L293D
- added D1, D2: (no value), SparkFun-LED:LED3MM
- added L298N: L293D, st-microelectronics:L293D
- added R1, R2: 220, resistor:R-US_0207/12
Connections:
- net N$10 renamed V
- new net N$1: R2.2, U$1.A7
- new net N$2: R1.2, U$1.D13
- new net N$3: D1.A, R1.1
- new net N$4: D2.A, R2.1
- net EN1-2: now also L298N.1-2EN; no longer L293D.1-2EN
- net EN3-4: now also L298N.3-4EN; no longer L293D.3-4EN
- net GND: now also D1.C, D2.C, L298N.GND1, L298N.GND2, L298N.GND3, L298N.GND4; no longer L293D.GND1, L293D.GND2, L293D.GND3, L293D.GND4
- net IN1: now also L298N.1A; no longer L293D.1A
- net IN2: now also L298N.2A; no longer L293D.2A
- net IN3: now also L298N.3A; no longer L293D.3A
- net IN4: now also L298N.4A; no longer L293D.4A
- net V+: now also L298N.VCC2; no longer L293D.VCC2
- net VCC: now also L298N.VCC1; no longer L293D.VCC1
- net VLEFT+: now also L298N.1Y; no longer L293D.1Y
- net VLEFT-: now also L298N.2Y; no longer L293D.2Y
- net VRIGHT+: now also L298N.4Y; no longer L293D.4Y
- net VRIGHT-: now also L298N.3Y; no longer L293D.3Y
Other:
- moved on the sheet: BATTERY, BLEUTOOTH, C1, C3, MOTOR-LEFT, MOTOR-RIGHT, QTR-MD-06, R3, R4, SHARP, SWITCH
